File: Ham_RF.sch (KiCad schematic (older format))
At the start: 88 parts, among them J1 SMA_EDGE, U10 SKY13388, U11 SKY13388, U4 TRF37A75, U7 TQP7M9105, U8 TQP7M9105, U9 TQP7M9105

Commit message: update to HS1.0b
Parts:
- removed C50: 1u, Capacitors_SMD:C_0402, symbol C-RESCUE-HAMShield04
- removed C52: 24p, Capacitors_SMD:C_0603, symbol C-RESCUE-HAMShield04
- removed C54: 43p, Capacitors_SMD:C_0603, symbol C-RESCUE-HAMShield04
- removed C57: 180p, Capacitors_SMD:C_0805, symbol C-RESCUE-HAMShield04
- removed C64: 10p, Capacitors_SMD:C_0402, symbol C-RESCUE-HAMShield04
- removed C65: 15p, Capacitors_SMD:C_0402, symbol C-RESCUE-HAMShield04
- removed L13: 5.6n, Capacitors_SMD:C_0603, symbol INDUCTOR_SMALL
- removed L14: 18n, Capacitors_SMD:C_0402, symbol INDUCTOR_SMALL
- removed L6, L7: 100n, Capacitors_SMD:C_0603, symbol INDUCTOR0603
- removed U7, U8: TQP7M9105, Housings_SOT-89:SOT89-3_Housing, symbol TQP7M9105
- added C48: 100p, Capacitors_SMD:C_0603, symbol C-RESCUE-HAMShield04
- added L6: 3.6n, Capacitors_SMD:C_0402, symbol INDUCTOR_SMALL
- added L7: 2n, Capacitors_SMD:C_0603, symbol INDUCTOR_SMALL
- added R5: 49.9, Resistors_SMD:R_0402, symbol RESISTOR0603-RES
- C26: value 1n -> 7p
- C27: value 1n -> 8p
- C32: value 0u1 -> 14p
- C33: value 0u1 -> 24p; footprint Capacitors_SMD:C_0402 -> Capacitors_SMD:C_0603
- C34: value 24p -> 11p; footprint Capacitors_SMD:C_0603 -> Capacitors_SMD:C_0402
- C38: value 56p -> 7p; footprint Capacitors_SMD:C_0603 -> Capacitors_SMD:C_0402
- C44: value 100p -> 47p; footprint Capacitors_SMD:C_0603 -> Capacitors_SMD:C_0402
- C45: value 15p -> 5.1p
- C46: value 1u -> 2.2p
- C49: value 43p -> 2.2p; footprint Capacitors_SMD:C_0603 -> Capacitors_SMD:C_0402
- C69: value 68p -> 15p; footprint Capacitors_SMD:C_0603 -> Capacitors_SMD:C_0402
- C72: value 27p -> 14p
- J1: footprint SMA-EDGE -> mogar_modules_new:SMA-EDGE-HandSolder
- L1: value 1ohm -> 5.6n; footprint Capacitors_SMD:C_0402 -> Capacitors_SMD:C_0603
- L11: value 6.2n -> 0ohm; footprint Capacitors_SMD:C_0603 -> Capacitors_SMD:C_0402
- L12: value 12n -> 6.2n; footprint Capacitors_SMD:C_0402 -> Capacitors_SMD:C_0603
- L15: footprint Capacitors_SMD:C_0603 -> mogar_modules_new:L_1008
- L16: value 12n -> 2n; footprint Capacitors_SMD:C_0402 -> Capacitors_SMD:C_0603
- L17: value 33n -> 3.3n; footprint Capacitors_SMD:C_0603 -> Capacitors_SMD:C_0402
- L4: value 15n -> 3.9n; footprint Capacitors_SMD:C_0603 -> Capacitors_SMD:C_0402
- L5: value 3.6n -> 3n; footprint Capacitors_SMD:C_0402 -> Capacitors_SMD:C_0603
- L8: value 3.6n -> 3.9n
- L9: value 24n -> 6.2n; footprint Capacitors_SMD:C_0402 -> Capacitors_SMD:C_0603
Connections:
- net GND: now also R5.1
- net STAGE1_OUT: now also C49.1, L9.1; no longer U11.11 (ANT)
- net VTX: now also C30.1, C37.1, C51.1, L15.2
- net at C45.1, L10.1: now also L12.2; no longer C23.2
- net at C38.1, L10.2: now also L8.1; no longer L1.1
- net at L1.2: now also C27.1, L4.1
- net at L8.2: now also C34.1, L6.1
- net at L9.2: now also C26.1, L1.1
- net S2_IN: now reaches U9.1 (RFin)
- net S2_IN: now also L11.2
- net at L16.2, U9.3 (RFout): now also L15.1; no longer L15.2
- net at C72.1, L17.1: now also L6.2; no longer L20.2
- net at L4.2, L5.1: now also C32.1; no longer C44.1
- net at L5.2: now also C33.1, L7.1
- net at L19.2: now also C24.2
- net at L11.1: now also C44.1, L7.2
- net at L18.2: now also C23.2; no longer L12.1
- net at U11.1 (RF1): now also R5.2
- removed net V_1.2M: C27.1, C33.1
- removed net V_2M: C30.1, C37.1, C51.1, L15.1
- removed net V_70CM: C26.1, C32.1, C46.1
- new net: C25.2, L20.2
- new net: C46.1, C48.1, L12.1
- new net STAGE2_OUT: C48.2, U11.11 (ANT)
- no-connect marks 1 -> 0
Other:
- moved on the sheet: C23, C24, C25, C49, C56, C58, C60, C61, C63, C66, C68, C70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
