File: PowerCtl.sch (KiCad schematic (older format))
At the start: 32 parts, among them Q1 NTGD1100L, Q2 NTGD1100L, Q3 NTGD1100L, Q4 NTGD1100L, U13 NC7SZ08, U14 NC7SZ08, U15 NC7SZ08, U2 MCP16311, U6 AP2125N-3.3TRG1

Commit message: update to HS1.0b
Parts:
- removed C47, C48, C55: 0u1, Capacitors_SMD:C_0402, symbol CAP0603-CAP
- removed Q2, Q3, Q4: NTGD1100L, mogar_modules_new:SC-74, symbol NTGD1100L
- removed R5, R6, R7: 10k, Resistors_SMD:R_0402, symbol R-RESCUE-HAMShield04
- removed U13, U14, U15: NC7SZ08, Transistors_SMD:sc70-5, symbol NC7SZ08
- U6: footprint TO_SOT_Packages_SMD:SOT-23_Handsoldering -> TO_SOT_Packages_SMD:SOT-23
Connections:
- net V1: now also D1.2 (A2); no longer D1.1 (A1)
- net V2: now also D1.1 (A1); no longer D1.2 (A2)
Other:
- note removed: "May want to choose MCP16312 for low noise"
- moved on the sheet: C16, C20, C22, C80, C81, D1, Q1, R4, U6
