File: UserInterface.sch (KiCad schematic (older format))
At the start: 31 parts, among them J2 SJ-43514-SMT-TR, Q5 BSS138, Q6 BSS138, Q7 BSS138, U3 AD8591, U5 ARDUINO_SHIELD

Commit message: update to HS1.0b
Parts:
- added C47: 2u2, Capacitors_SMD:C_0603, symbol CAP0603-CAP
- added D2, D3: LED, Diodes_SMD:D_0603, symbol LED
- added R20, R22: 330, Resistors_SMD:R_0402, symbol RESISTOR0603-RES
- added R6, R7: 10k, Resistors_SMD:R_0402, symbol RESISTOR0603-RES
- C41: value 1n -> 15n
- C42: value 0u1 -> 2u2; footprint Capacitors_SMD:C_0402 -> Capacitors_SMD:C_0603
- C93: value 0u1 -> 47u; footprint Capacitors_SMD:C_0402 -> mogar_modules_new:C1210P
- JP3: footprint SparkFun:SparkFun-1X04 -> Pin_Headers:Pin_Header_Straight_1x04_Pitch2.54mm
- Q5, Q6, Q7: footprint TO_SOT_Packages_SMD:SOT-23_Handsoldering -> TO_SOT_Packages_SMD:SOT-23
- R12: value dnp -> 10k
- R13: value 0 -> 10k
- R24: value 20k -> 1.47k
- U5: footprint mogar_modules_new:ARDUINO_SHIELD -> mogar_modules_new:ARDUINO_UNO_SHIELD
Connections:
- net AFOUT: now also C47.1; no longer U3.3 (+IN)
- net GND: now also D2.1 (K), D3.1 (K), R7.2; no longer R12.1
- net VCC: now also R12.1, R22.1
- net VTX: now also R20.1
- net at R13.1, U3.4 (-IN): now also R6.2; no longer R12.2
- new net: R12.2, R7.1, U3.3 (+IN)
- new net: D2.2 (A), R20.2
- new net: D3.2 (A), R22.2
- new net: C47.2, R6.1
Other:
- note added: "Gain = (Rf/Ri) = 2"
- note added: "Power LED"
- note added: "TX LED"
- note removed: "Gain = (1+Rf/Rg) = 1"
- moved on the sheet: Q5, Q6, Q7, R1, R12, R14, R15, R16, R17, R2, R3, R36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
